Commit message: fixed problem with urdf macro with joint limited

File: ur5_robotiq_arg140_description/robots/ur5_robotiq_140_joint_limited.xacro (robot description, xacro)
@@ -7,5 +7,5 @@
   <xacro:macro name="ur5_with_gripper_joint_limited" params="prefix">
     <!-- arm -->
-    <xacro:ur5_robot prefix="${prefix}ur5_" joint_limited="true"
+    <xacro:ur5_robot prefix="${prefix}" joint_limited="true"
       shoulder_pan_lower_limit="${-pi}" shoulder_pan_upper_limit="${pi}"
       shoulder_lift_lower_limit="${-pi}" shoulder_lift_upper_limit="${pi}"
@@ -16,14 +16,14 @@
     />
     <!-- gripper -->
-    <xacro:robotiq_arg2f_140 prefix="${prefix}gripper_" />
+    <xacro:robotiq_arg2f_140 prefix="${prefix}" />
     <link name="${prefix}world" />
     <joint name="world_joint" type="fixed">
       <parent link= "${prefix}world" />
-      <child link = "${prefix}ur5_base_link" />
+      <child link = "${prefix}base_link" />
       <origin xyz="0.0 0.0 0.0" rpy="0.0 0.0 0.0" />
     </joint>
     <joint name="ur5_tool0-gripper_base" type="fixed">
-      <parent link= "${prefix}ur5_tool0" />
-      <child link = "${prefix}gripper_robotiq_arg2f_base_link" />
+      <parent link= "${prefix}tool0" />
+      <child link = "${prefix}robotiq_arg2f_base_link" />
       <origin xyz="0.0 0.0 0.0" rpy="0.0 0.0 0.0" />
     </joint>
