Commit message: bug fixes

File: ur5_robotiq_arg140_description/robots/robotiq_arg140_description_macro.xacro (robot description, xacro)
@@ -167,14 +167,14 @@
         <origin xyz="0 0 0" rpy="0 0 0" />
         <geometry>
-          <mesh filename="package://ur5_robotiq_arg140_description/meshes/finger_tip.stl" />
-        </geometry>
-        <material name="">
-          <color rgba="0.1 0.1 0.1 1" />
-        </material>
-      </visual>
-      <collision>
-        <origin xyz="0 0 0" rpy="0 0 0" />
-        <geometry>
-          <mesh filename="package://ur5_robotiq_arg140_description/meshes/finger_tip.stl" />
+          <mesh filename="package://ur5_robotiq_arg140_description/meshes/finger_tip.dae" />
+        </geometry>
+        <material name="">
+          <color rgba="0.1 0.1 0.1 1" />
+        </material>
+      </visual>
+      <collision>
+        <origin xyz="0 0 0" rpy="0 0 0" />
+        <geometry>
+          <mesh filename="package://ur5_robotiq_arg140_description/meshes/finger_tip.d" />
         </geometry>
       </collision>

File: ur5_robotiq_arg140_description/urdf/robotiq_arg2f.xacro (robot description, xacro)
@@ -1,5 +1,5 @@
 <?xml version="1.0"?>
 <robot xmlns:xacro="http://ros.org/wiki/xacro">
-  <xacro:include filename="$(find ur5_robotiq_arg140_description)/urdf/robotiq_arg2f_finger_tips.xacro" />
+  <!--xacro:include filename="$(find ur5_robotiq_arg140_description)/urdf/robotiq_arg2f_finger_tips.xacro" /-->
   <xacro:macro name="robotiq_arg2f_base_link" params="prefix">
     <link name="${prefix}robotiq_arg2f_base_link">

File: ur5_robotiq_arg140_description/urdf/robotiq_arg2f_140_model_macro.xacro (robot description, xacro)
@@ -150,5 +150,4 @@
     </joint>
   </xacro:macro>
-  <xacro:include filename="$(find ur5_robotiq_arg140_description)/urdf/robotiq_arg2f.xacro" />
   <xacro:macro name="finger_joint" params="prefix">
     <joint name="${prefix}finger_joint" type="revolute">
@@ -172,4 +171,45 @@
     <xacro:finger_joints prefix="${prefix}" fingerprefix="right" reflect="-1.0"/>
   </xacro:macro>
+  <!--finger tip-->
+  <xacro:macro name="finger_tip" params="prefix fingerprefix stroke">
+    <link name="${prefix}${fingerprefix}_finger_tip">
+      <inertial>
+        <origin xyz="0.000299999999999317 0.0160078233491243 -0.0136945669206257" rpy="0 0 0" />
+        <mass value="0.0104003125914103" />
+        <inertia
+            ixx="2.71909453810972E-06"
+            ixy="0.0"
+            ixz="0.0"
+            iyy="7.69100314106116E-07"
+            iyz="0.0"
+            izz="2.30315190420171E-06" />
+      </inertial>
+      <visual>
+        <origin xyz="0 0 0" rpy="0 0 0" />
+        <geometry>
+          <mesh filename="package://ur5_robotiq_arg140_description/meshes/robotiq_arg2f_${stroke}_finger_tip.dae" />
+        </geometry>
+        <material name="">
+          <color rgba="0.1 0.1 0.1 1" />
+        </material>
+      </visual>
+      <collision>
+        <origin xyz="0 0 0" rpy="0 0 0" />
+        <geometry>
+          <mesh filename="package://ur5_robotiq_arg140_description/meshes/robotiq_arg2f_${stroke}_finger_tip.dae" />
+        </geometry>
+      </collision>
+    </link>
+  </xacro:macro>
+  <xacro:macro name="finger_tip_joint" params="prefix fingerprefix">
+    <joint name="${prefix}${fingerprefix}_finger_tip_joint" type="fixed">
+      <origin xyz="0 0.01821998610742 0.0260018192872234" rpy="0 0 0" />
+      <parent link="${prefix}${fingerprefix}_inner_finger" />
+      <child link="${prefix}${fingerprefix}_finger_tip" />
+      <axis xyz="1 0 0" />
+    </joint>
+  </xacro:macro>
+    <!--Import robotiq desciptions-->
+  <xacro:include filename="$(find ur5_robotiq_arg140_description)/urdf/robotiq_arg2f.xacro" />
   <xacro:macro name="robotiq_arg2f_140" params="prefix">
     <xacro:robotiq_arg2f_base_link prefix="${prefix}"/>

File: ur5_robotiq_arg140_description/urdf/robotiq_arg2f_finger_tips.xacro (robot description, xacro)
@@ -17,5 +17,5 @@
         <origin xyz="0 0 0" rpy="0 0 0" />
         <geometry>
-          <mesh filename="package://ur5_robotiq_arg140_description/meshes/robotiq_arg2f_${stroke}_finger_tip.stl" />
+          <mesh filename="package://ur5_robotiq_arg140_description/meshes/robotiq_arg2f_${stroke}_finger_tip.dae" />
         </geometry>
         <material name="">
@@ -26,5 +26,5 @@
         <origin xyz="0 0 0" rpy="0 0 0" />
         <geometry>
-          <mesh filename="package://ur5_robotiq_arg140_description/meshes/robotiq_arg2f_${stroke}_inner_finger.stl" />
+          <mesh filename="package://ur5_robotiq_arg140_description/meshes/robotiq_arg2f_${stroke}_finger_tip.dae" />
         </geometry>
       </collision>
