Commit message: Bug fixes

File: icl_phri_ur5_robotiq_arg140_description/robots/ur5_robotiq_140.xacro (robot description, xacro)
@@ -5,5 +5,6 @@
   <xacro:include filename="$(find ur_description)/urdf/ur5.urdf.xacro" />
   <xacro:include filename="$(find icl_phri_ur5_robotiq_arg140_description)/urdf/robotiq_arg2f_140_model_macro.xacro" />
-  <xacro:macro name="ur5_with_gripper" params="prefix">
+  <xacro:include filename="$(find robotiq_force_torque_sensor)/urdf/robotiq_fts300.urdf.xacro" />
+  <xacro:macro name="ur5_with_gripper_joint_limited" params="prefix">
     <!-- arm -->
     <xacro:ur5_robot prefix="${prefix}" joint_limited="false" />
@@ -17,8 +18,12 @@
       <origin xyz="0.0 0.0 0.0" rpy="0.0 0.0 0.0" />
     </joint>
+    <!--force torque sensor-->
+    <xacro:robotiq_fts150 prefix="" parent="ee_link" >
+      <origin xyz="0 0 0" rpy="0 1.57 0"/>
+    </xacro:robotiq_fts150>
     <joint name="ur5_ee_link-gripper_base" type="fixed">
-      <parent link= "${prefix}ee_link" />
+      <parent link= "${prefix}fts_toolside" />
       <child link = "${prefix}robotiq_arg2f_base_link" />
-      <origin xyz=" 0.04 0.0 0.0" rpy="0.0 ${pi/2} 0.0" />
+      <origin xyz=" 0.0 0.0 0.0" rpy="0.0 0.0 0.0" />
     </joint>
     <link name="${prefix}tool" />
@@ -29,5 +34,5 @@
     </joint>
   </xacro:macro>
-  <xacro:ur5_with_gripper prefix=""/>
+  <xacro:ur5_with_gripper_joint_limited prefix=""/>
  <!-- Plugin -->
   <gazebo>

File: icl_phri_ur5_robotiq_arg140_description/robots/ur5_robotiq_140_joint_limited.xacro (robot description, xacro)
@@ -13,5 +13,5 @@
       elbow_joint_lower_limit="${-pi}" elbow_joint_upper_limit="${pi}"
       wrist_1_lower_limit="${-pi}" wrist_1_upper_limit="${pi}"
-      wrist_2_lower_limit="${-pi/2}" wrist_2_upper_limit="${pi/2}"
+      wrist_2_lower_limit="${-pi}" wrist_2_upper_limit="${pi}"
       wrist_3_lower_limit="${-pi}" wrist_3_upper_limit="${pi}"
     />
