Commit message: add gazebo simulation

File: icl_phri_ur5_robotiq_arg140_description/robots/ur5_robotiq_140_joint_limited_new.xacro (robot description, xacro)
@@ -5,5 +5,5 @@
   <xacro:include filename="$(find ur_description)/urdf/ur5.urdf.xacro" />
   <xacro:include filename="$(find icl_phri_ur5_robotiq_arg140_description)/urdf/robotiq_arg2f_140_model_macro.xacro" />
-  <xacro:include filename="$(find robotiq_force_torque_sensor)/urdf/robotiq_fts300.urdf.xacro" />
+  <link name="world"/>
   <xacro:macro name="ur5_with_gripper_joint_limited" params="prefix">
     <!-- arm -->
@@ -16,30 +16,17 @@
       wrist_3_lower_limit="${-pi}" wrist_3_upper_limit="${pi}"
     />
+	<joint name="ur5_world_joint" type="fixed">
+		<parent link="world" />
+		<child link = "${prefix}base_link" />
+		<origin xyz="0.0 0.0 0.0" rpy="0.0 0.0 0.0" />
+	</joint>
     <!-- gripper -->
     <xacro:robotiq_arg2f_140 prefix="${prefix}" />
-    <!--dummy link-->
-  	<link name="world" />
-    <joint name="fixed_link-robot_base" type="fixed">
-      <parent link= "world" />
-      <child link = "${prefix}base_link" />
-      <origin xyz="0.0 0.0 0.0" rpy="0.0 0.0 0.0" />
-    </joint>
-    <!--force torque sensor-->
-    <xacro:robotiq_fts150 prefix="" parent="ee_link" >
-      <origin xyz="0.009 0 0 " rpy="-${pi/2} 0 -${pi/2}"/>
-    </xacro:robotiq_fts150>
     <joint name="ur5_ee_link-gripper_base" type="fixed">
-      <parent link= "${prefix}fts_toolside" />
+      <parent link= "${prefix}ee_link" />
       <child link = "${prefix}robotiq_arg2f_base_link" />
-      <origin xyz=" 0.0 0.0 0.0" rpy="0.0 0.0 ${pi/2}" />
-    </joint>
-    <link name="${prefix}tool" />
-    <joint name="tool_tip" type="fixed">
-      <parent link= "${prefix}ee_link" />
-      <child link = "${prefix}tool" />
-      <origin xyz=" 0.00 0.0 0.1" rpy="0.0 0.0 0.0" />
+      <origin xyz=" 0.07 0.0 0.0" rpy="0.0 ${pi/2} 0" />
     </joint>
   </xacro:macro>
   <xacro:ur5_with_gripper_joint_limited prefix=""/>
- <!-- Plugin -->
 </robot>

File: icl_phri_ur5_robotiq_arg140_description/urdf/robotiq_arg2f_140_model_macro.xacro (robot description, xacro)
@@ -136,5 +136,6 @@
       <child link="${prefix}${fingerprefix}_inner_knuckle" />
       <axis xyz="1 0 0" />
-      <limit lower="0" upper="0.8757" velocity="2.0" effort="1000" />
+      <!--<limit lower="0" upper="0.8757" velocity="2.0" effort="1000" /> -->
+	  <limit lower="-3.14159" upper="3.14159" velocity="2.0" effort="1000" />
       <mimic joint="${prefix}finger_joint" multiplier="-1" offset="0" />
     </joint>
@@ -146,5 +147,6 @@
       <child link="${prefix}${fingerprefix}_inner_finger" />
       <axis xyz="1 0 0" />
-      <limit lower="0" upper="0.8757" velocity="2.0" effort="1000" />
+      <limit lower="-3.14159" upper="3.14159" velocity="2.0" effort="1000" />
+      <!-- <limit lower="0" upper="0.8757" velocity="2.0" effort="1000" /> -->
       <mimic joint="${prefix}finger_joint" multiplier="1" offset="0" />
     </joint>
@@ -156,4 +158,5 @@
       <child link="${prefix}left_outer_knuckle" />
       <axis xyz="-1 0 0" />
+      <!-- <limit lower="-3.14159" upper="3.14159" velocity="2.0" effort="1000" /> -->
       <limit lower="0" upper="0.775" velocity="2.0" effort="1000" />
     </joint>
@@ -166,5 +169,6 @@
       <child link="${prefix}right_outer_knuckle" />
       <axis xyz="1 0 0" />
-      <limit lower="0" upper="0.725" velocity="2.0" effort="1000" />
+      <!-- <limit lower="0" upper="0.725" velocity="2.0" effort="1000" /> -->
+	  <limit lower="-3.14159" upper="3.14159" velocity="2.0" effort="1000" />
     <mimic joint="${prefix}finger_joint" multiplier="-1" offset="0" />
     </joint>

File: icl_phri_ur5_robotiq_arg140_description/urdf/robotiq_arg2f_transmission.xacro (robot description, xacro)
@@ -11,4 +11,33 @@
       </actuator>
     </transmission>
+	    <gazebo>
+             <!-- loading plugin: mimic joints works in gazebo now-->
+             <plugin filename="libroboticsgroup_gazebo_mimic_joint_plugin.so" name="${prefix}mimic_robotiq_140_4">
+                <joint>${prefix}finger_joint</joint>
+                <mimicJoint>${prefix}right_outer_knuckle_joint</mimicJoint>
+                <multiplier>-1.0</multiplier>
+            </plugin>
+            <plugin filename="libroboticsgroup_gazebo_mimic_joint_plugin.so" name="${prefix}mimic_robotiq_140_2">
+                <joint>${prefix}finger_joint</joint>
+                <mimicJoint>${prefix}left_inner_finger_joint</mimicJoint>
+                <multiplier>1.0</multiplier>
+                <!--<offset>0.0</offset>-->
+            </plugin>
+            <plugin filename="libroboticsgroup_gazebo_mimic_joint_plugin.so" name="${prefix}mimic_robotiq_140_1">
+                <joint>${prefix}finger_joint</joint>
+                <mimicJoint>${prefix}right_inner_finger_joint</mimicJoint>
+                <multiplier>1.0</multiplier>
+            </plugin>
+            <plugin filename="libroboticsgroup_gazebo_mimic_joint_plugin.so" name="${prefix}mimic_robotiq_140_3">
+                <joint>${prefix}finger_joint</joint>
+                <mimicJoint>${prefix}left_inner_knuckle_joint</mimicJoint>
+                <multiplier>-1.0</multiplier>
+            </plugin>
+            <plugin filename="libroboticsgroup_gazebo_mimic_joint_plugin.so" name="${prefix}mimic_robotiq_140_5">
+                <joint>${prefix}finger_joint</joint>
+                <mimicJoint>${prefix}right_inner_knuckle_joint</mimicJoint>
+                <multiplier>-1.0</multiplier>
+            </plugin>
+        </gazebo>
   </xacro:macro>
 </robot>
